Commit message: fixed the orientation of the tool in urdf

File: src/iiwa_stack_examples/iiwa_tool/iiwa_tool_description/urdf/iiwa_tool.urdf.xacro (robot description, xacro)
@@ -45,5 +45,6 @@
     <parent link="iiwa_link_ee" />
     <child link = "tool_link" />
-    <origin xyz="${tool_joint_offset}" rpy="0 ${PI/2.0} 0" />
+    <!-- <origin xyz="${tool_joint_offset}" rpy="0 ${PI/2.0} 0" />   -->
+    <origin xyz="${tool_joint_offset}" rpy="0 0 0" />
   </joint>
   <!-- Here we define the geometry of the tool. We designed the tool ourselves, so we have a mesh file that represents it.
